File: plain60-flex-edition.kicad_pcb (KiCad board)
At the start: 2 copper layers, 284.7 x 94.2 mm, 175 parts, among them J1 HRO-TYPE-C-31-M-12, J2 ISP, J3 ai03_ud, K1 KEYSW, K10 KEYSW, K11 KEYSW, K12 KEYSW, K13 KEYSW, K14 KEYSW, K15 KEYSW, K15-1 KEYSW, K16 KEYSW, K17 KEYSW, K18 KEYSW, K19 KEYSW, K2 KEYSW, K20 KEYSW, K21 KEYSW, K22 KEYSW, K23 KEYSW, K24 KEYSW, K25 KEYSW, K26 KEYSW, K27 KEYSW, K28 KEYSW, K29 KEYSW, K3 KEYSW, K31 KEYSW, K31-1 KEYSW, K32 KEYSW, K33 KEYSW, K34 KEYSW, K35 KEYSW, K36 KEYSW, K37 KEYSW, K38 KEYSW, K39 KEYSW, K4 KEYSW, K40 KEYSW, K41 KEYSW, K42 KEYSW, K43 KEYSW, K44 KEYSW, K44-1 KEYSW, K46 KEYSW, K46-1 KEYSW, K47 KEYSW, K48 KEYSW, K49 KEYSW, K5 KEYSW, K50 KEYSW, K51 KEYSW, K52 KEYSW, K53 KEYSW, K54 KEYSW, K55 KEYSW, K56 KEYSW, K57 KEYSW, K58 KEYSW, K58-1 KEYSW, K59 KEYSW, K6 KEYSW, K61 KEYSW, K61-1 KEYSW, K62 KEYSW, K62-1 KEYSW, K63 KEYSW, K63-1 KEYSW, K67 KEYSW, K67-1 KEYSW, K7 KEYSW, K71 KEYSW, K72 KEYSW, K72-1 KEYSW, K73 KEYSW, K73-1 KEYSW, K74 KEYSW, K74-1 KEYSW, K8 KEYSW, K9 KEYSW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

Commit message: removed ansi and 6.25u support
Parts:
- removed D14, D29, D71: D, Keeb_components:D_0805
- removed K14, K15-1: KEYSW, Keeb_switches:CHERRY_PLATE_100H
- removed K29: KEYSW, Keeb_switches:CHERRY_PLATE_150H
- removed K44: KEYSW, Keeb_switches:CHERRY_PCB_225H_F
- removed K46: KEYSW, Keeb_switches:CHERRY_PCB_225H
- removed K61, K62, K63, K71, K72, K73, K74: KEYSW, Keeb_switches:CHERRY_PLATE_125H
- removed K67: KEYSW, Keeb_switches:CHERRY_PCB_625H_F
- removed LS1: Speaker, Keeb_components:speaker_AST1109MLTRQ
- moved D44 11.9 mm to (262.9, 41.2)
Connections:
- K15 pad 1: col14 -> col13
Routing:
- net col14: track 313.1 -> 0.00 mm, vias 1 -> 0
- net Net-(LS1-Pad1): track 187.3 -> 0.00 mm, vias 2 -> 0
- net GND: track 245.5 -> 62.0 mm, vias 22 -> 20
- net col10: track 399.1 -> 322.4 mm
- net Net-(D29-Pad2): track 37.2 -> 0.00 mm
- net Net-(D67-Pad2): track 19.2 -> 7.30 mm
- net Net-(D15-Pad2): track 29.4 -> 19.9 mm
- net col0: track 128.6 -> 119.1 mm
- net Net-(D71-Pad2): track 7.30 -> 0.00 mm
- net Net-(D44-Pad2): track 15.6 -> 8.97 mm
- net row2: track 243.5 -> 238.0 mm
- net Net-(D14-Pad2): track 4.98 -> 0.00 mm
- net col13: track 355.6 -> 350.7 mm
- net row0: track 276.0 -> 272.4 mm
- net Net-(D62-Pad2): track 15.6 -> 13.3 mm
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Other:
- outline, holes or cut-outs redrawn
- board text removed: "Speaker AST1109MLTRQ Pin B7"
